File: ESP32-WROOM.sch (KiCad schematic (older format))
At the start: 4 parts

Commit message: Added annotations to the ESP32 sheet to make clear which I/O are used in UART programming.
Other:
- note added: "These pins are used for programming in UART mode."
- note added: "This pin is used for selecting boot mode."
- note added: "Use of these\npins is not\nrecommended."
Changed lines of the file:
@@
 	4100 3050 4050 3050
 Connection ~ 4100 3050
+Text Notes 5150 5100 0    50   ~ 0
+Use of these\npins is not\nrecommended.
+Wire Notes Line
+	5100 5100 5700 5100
+Wire Notes Line
+	5700 5100 5700 4600
+Wire Notes Line
+	5100 4600 5100 5100
+Text Notes 6500 4300 0    50   ~ 0
+This pin is used for selecting boot mode.
+Text Notes 6600 3300 0    50   ~ 0
+These pins are used for programming in UART mode.
+Wire Notes Line
+	8150 4200 8150 4350
+Wire Notes Line
+	6450 4200 8150 4200
+Wire Notes Line
+	6450 4350 8150 4350
+Wire Notes Line
+	8650 3200 8650 3400
+Wire Notes Line
+	8650 3400 6450 3400
+Wire Notes Line
+	6450 3200 8650 3200
 $EndSCHEMATC

Commit message: Annotated schematic and added footprints.
Parts:
- C4: renamed from C?; footprint (none) -> Capacitors_SMD:C_1210
- C5: renamed from C?; footprint (none) -> Capacitors_SMD:C_0603
- R8: renamed from R?; footprint (none) -> Resistors_SMD:R_0603
- gave numbers to parts that had none: 1
Changed lines of the file:
@@
 $EndDescr
 $Comp
-L ESP32-footprints-Shem-Lib:ESP32-WROOM U?
+L ESP32-footprints-Shem-Lib:ESP32-WROOM U2
 U 1 1 5BD760E7
 P 5400 3550
-F 0 "U?" H 5375 4937 60  0000 C CNN
+F 0 "U2" H 5375 4937 60  0000 C CNN
 F 1 "ESP32-WROOM" H 5375 4831 60  0000 C CNN
 F 2 "ESP32-footprints-Lib:ESP32-WROOM" H 5750 4900 60  0001 C CNN
@@
 	4950 4750 4950 4600
 $Comp
-L Device:R R?
+L Device:R R8
 U 1 1 5BD77283
 P 4100 2850
-F 0 "R?" H 4170 2896 50  0000 L CNN
+F 0 "R8" H 4170 2896 50  0000 L CNN
 F 1 "10kR" H 4170 2805 50  0000 L CNN
-F 2 "" V 4030 2850 50  0001 C CNN
+F 2 "Resistors_SMD:R_0603" V 4030 2850 50  0001 C CNN
 F 3 "~" H 4100 2850 50  0001 C CNN
 	1    4100 2850
@@
 NoConn ~ 6300 3550
 $Comp
-L Device:C C?
+L Device:C C5
 U 1 1 5BD8BBC9
 P 3450 2300
-F 0 "C?" H 3565 2346 50  0000 L CNN
+F 0 "C5" H 3565 2346 50  0000 L CNN
 F 1 "0.1uF" H 3565 2255 50  0000 L CNN
-F 2 "" H 3488 2150 50  0001 C CNN
+F 2 "Capacitors_SMD:C_0603" H 3488 2150 50  0001 C CNN
 F 3 "~" H 3450 2300 50  0001 C CNN
 	1    3450 2300
@@
 $EndComp
 $Comp
-L Device:CP C?
+L Device:CP C4
 U 1 1 5BD8BC61
 P 2950 2300
-F 0 "C?" H 3068 2346 50  0000 L CNN
+F 0 "C4" H 3068 2346 50  0000 L CNN
 F 1 "100uF" H 3068 2255 50  0000 L CNN
-F 2 "" H 2988 2150 50  0001 C CNN
+F 2 "Capacitors_SMD:C_1210" H 2988 2150 50  0001 C CNN
 F 3 "~" H 2950 2300 50  0001 C CNN
 	1    2950 2300
